Commit message: complete ass1 model, begin ass4 file

File: URDF/MDaK_assignment_4.urdf (robot description, URDF)
Before this commit: robot franka_research_3, 29 links, 28 joints
Links:
- removed link arm_link_1a
- removed link arm_link_1b
- removed link arm_link_1c
- removed link arm_link_2a
- removed link arm_link_2b
- removed link arm_link_2c
- removed link arm_link_3a
- removed link arm_link_3b
- removed link arm_link_3c
- removed link arm_link_3d
- removed link arm_link_3e
- removed link arm_link_4a
- removed link arm_link_4b
- removed link arm_link_4c
- removed link arm_link_4d
- removed link arm_link_4e
- removed link arm_link_5a
- removed link arm_link_5b
- removed link arm_link_5c
- removed link arm_link_5d
- removed link arm_link_6a
- removed link arm_link_6b
- removed link arm_link_6c
- removed link arm_link_7a
- removed link arm_link_7b
- removed link arm_link_7c
- removed link base_box
- removed link base_cyl
Joints:
- removed joint arm_link_1a_to_base_cyl
- removed joint arm_link_1b_to_1a
- removed joint arm_link_1c_to_1b
- removed joint arm_link_2a_to_2b
- removed joint arm_link_2b_to_1b
- removed joint arm_link_2c_to_2b
- removed joint arm_link_3a_to_2a
- removed joint arm_link_3b_to_3a
- removed joint arm_link_3c_to_3a
- removed joint arm_link_3d_to_3b
- removed joint arm_link_3e_to_3b
- removed joint arm_link_4a_to_4b
- removed joint arm_link_4b_to_3b
- removed joint arm_link_4c_to_4a
- removed joint arm_link_4d_to_4b
- removed joint arm_link_4e_to_4b
- removed joint arm_link_5a_to_4a
- removed joint arm_link_5b_to_5a
- removed joint arm_link_5c_to_5a
- removed joint arm_link_5d_to_5a
- removed joint arm_link_6a_to_6b
- removed joint arm_link_6b_to_5b
- removed joint arm_link_6c_to_6b
- removed joint arm_link_7a_to_6a
- removed joint arm_link_7b_to_7a
- removed joint arm_link_7c_to_7a
- removed joint base_box_to_world
- removed joint base_cyl_to_base_box

Commit message: trying xacro and pybullet commands

File: URDF/MDaK_assignment_4.urdf (robot description, URDF)
Before this commit: robot poolbot, 1 links, 0 joints
Links:
- added link table_leg_FL; visual cylinder length=0.5 radius=0.075
Joints:
- added joint table_leg_FL_to_world: type fixed, parent world, child table_leg_FL, origin xyz=1 ${tablewidth/2} 0
