Commit message: Update pool_bot.xacro

File: URDF/pool_bot.xacro (robot description, xacro)
@@ -1 +1,46 @@
 <?xml version="1.0"?>
+<robot xmlns:xacro="http://www.ros.org/wiki/xacro" name="pool_table">
+  <!-- Define Parameters -->
+  <xacro:property name="table_leg_radius" value="0.075"/>
+  <xacro:property name="table_leg_length" value="0.5"/>
+  <xacro:property name="table_inner_width" value="0.82"/>
+  <!-- Define macro for table legs -->
+  <xacro:macro name="table_leg" params="name">
+    <link name="table_leg_${name}">
+      <visual>
+        <geometry>
+          <cylinder radius="${table_leg_radius}" length="${table_leg_length}"/>
+        </geometry>
+        <origin xyz="0 0 ${table_leg_length/2}"/>
+        <material name="brown"/>
+      </visual>
+      <collision>
+        <geometry>
+          <cylinder radius="${table_leg_radius}" length="${table_leg_length}"/>
+        </geometry>
+        <origin xyz="0 0 ${table_leg_length/2}"/>
+      </collision>
+    </link>
+  </xacro:macro>
+  <!-- Define Materials -->
+  <material name="black">
+    <color rgba="0 0 0 1"/>
+  </material>
+  <material name="white">
+    <color rgba="1 1 1 1"/>
+  </material>
+  <material name="brown">
+    <color rgba="0.56 0.32 0.12 1"/>
+  </material>
+  <!-- Define links and joints -->
+  <link name="world">
+  </link>
+  <xacro:table_leg name="FL"/>
+  <xacro:table_leg name="BL"/>
+  <xacro:table_leg name="FR"/>
+  <xacro:table_leg name="BR"/>
+  <joint name="table_leg_FL_to_world" type="fixed">
+    <parent link="world"/>
+    <child link="table_leg_FL"/>
+    <origin xyz="1 ${tablewidth/2} 0"/>
+  </joint>

Commit message: Update pool_bot.xacro

File: URDF/pool_bot.xacro (robot description, xacro)
@@ -5,4 +5,9 @@
   <xacro:property name="table_leg_length" value="0.5"/>
   <xacro:property name="table_inner_width" value="0.82"/>
+  <xacro:property name="table_outer_width" value="1.12"/>
+  <xacro:property name="table_inner_length" value="1.6"/>
+  <xacro:property name="table_outer_length" value="1.9"/>
+  <xacro:property name="table_inner_height" value="0.75"/>
+  <xacro:property name="table_outer_height" value="0.8"/>
   <!-- Define macro for table legs -->
   <xacro:macro name="table_leg" params="name">
@@ -43,4 +48,22 @@
     <parent link="world"/>
     <child link="table_leg_FL"/>
-    <origin xyz="1 ${tablewidth/2} 0"/>
+    <origin xyz="${3*table_inner_length/8} ${3*table_inner_width/8} 0"/>
   </joint>
+  <joint name="table_leg_BL_to_world" type="fixed">
+    <parent link="world"/>
+    <child link="table_leg_BL"/>
+    <origin xyz="${-3*table_inner_length/8} ${3*table_inner_width/8} 0"/>
+  </joint>
+  <joint name="table_leg_FR_to_world" type="fixed">
+    <parent link="world"/>
+    <child link="table_leg_FR"/>
+    <origin xyz="${3*table_inner_length/8} ${-3*table_inner_width/8} 0"/>
+  </joint>
+  <joint name="table_leg_BR_to_world" type="fixed">
+    <parent link="world"/>
+    <child link="table_leg_BR"/>
+    <origin xyz="${-3*table_inner_length/8} ${-3*table_inner_width/8} 0"/>
+  </joint>
+  <!-- Tabletop (CAD?)
+    <link name="
+  -->

Commit message: try to use xacro

File: URDF/pool_bot.xacro (robot description, xacro)
@@ -48,20 +48,20 @@
     <parent link="world"/>
     <child link="table_leg_FL"/>
-    <origin xyz="${3*table_inner_length/8} ${3*table_inner_width/8} 0"/>
+    <origin xyz="${3*table_inner_width/8} ${3*table_inner_length/8} 0"/>
   </joint>
   <joint name="table_leg_BL_to_world" type="fixed">
     <parent link="world"/>
     <child link="table_leg_BL"/>
-    <origin xyz="${-3*table_inner_length/8} ${3*table_inner_width/8} 0"/>
+    <origin xyz="${-3*table_inner_width/8} ${3*table_inner_length/8} 0"/>
   </joint>
   <joint name="table_leg_FR_to_world" type="fixed">
     <parent link="world"/>
     <child link="table_leg_FR"/>
-    <origin xyz="${3*table_inner_length/8} ${-3*table_inner_width/8} 0"/>
+    <origin xyz="${3*table_inner_width/8} ${-3*table_inner_length/8} 0"/>
   </joint>
   <joint name="table_leg_BR_to_world" type="fixed">
     <parent link="world"/>
     <child link="table_leg_BR"/>
-    <origin xyz="${-3*table_inner_length/8} ${-3*table_inner_width/8} 0"/>
+    <origin xyz="${-3*table_inner_width/8} ${-3*table_inner_length/8} 0"/>
   </joint>
   <!-- Tabletop (CAD?)

Commit message: Update pool_bot and get xacro working

File: URDF/pool_bot.xacro (robot description, xacro)
@@ -17,5 +17,5 @@
           <cylinder radius="${table_leg_radius}" length="${table_leg_length}"/>
         </geometry>
-        <origin xyz="0 0 ${table_leg_length/2}"/>
+        <origin xyz="0 0 -${table_leg_length/2}"/>
         <material name="brown"/>
       </visual>
@@ -24,5 +24,5 @@
           <cylinder radius="${table_leg_radius}" length="${table_leg_length}"/>
         </geometry>
-        <origin xyz="0 0 ${table_leg_length/2}"/>
+        <origin xyz="0 0 -${table_leg_length/2}"/>
       </collision>
     </link>
@@ -41,29 +41,47 @@
   <link name="world">
   </link>
+  <link name="tabletop">
+    <visual>
+      <geometry>
+        <box size="${table_outer_width} ${table_outer_length} ${table_inner_height-table_leg_length}"/>
+      </geometry>
+      <origin xyz="0 0 ${(table_inner_height-table_leg_length)/2}"/>
+      <material name="brown"/>
+    </visual>
+    <collision>
+      <geometry>
+        <box size="${table_outer_width} ${table_outer_length} ${table_inner_height-table_leg_length}"/>
+      </geometry>
+      <origin xyz="0 0 ${(table_inner_height-table_leg_length)/2}"/>
+    </collision>
+  </link>
+  <joint name="tabletop_to_world" type="fixed">
+    <parent link="world"/>
+    <child link="tabletop"/>
+    <origin xyz="0 0 ${table_leg_length}"/>
+  </joint>
   <xacro:table_leg name="FL"/>
   <xacro:table_leg name="BL"/>
   <xacro:table_leg name="FR"/>
   <xacro:table_leg name="BR"/>
-  <joint name="table_leg_FL_to_world" type="fixed">
-    <parent link="world"/>
+  <joint name="table_leg_FL_to_tabletop" type="fixed">
+    <parent link="tabletop"/>
     <child link="table_leg_FL"/>
-    <origin xyz="${3*table_inner_width/8} ${3*table_inner_length/8} 0"/>
+    <origin xyz="${table_inner_width/2} ${table_inner_length/2} 0"/>
   </joint>
-  <joint name="table_leg_BL_to_world" type="fixed">
-    <parent link="world"/>
+  <joint name="table_leg_BL_to_tabletop" type="fixed">
+    <parent link="tabletop"/>
     <child link="table_leg_BL"/>
-    <origin xyz="${-3*table_inner_width/8} ${3*table_inner_length/8} 0"/>
+    <origin xyz="${-table_inner_width/2} ${table_inner_length/2} 0"/>
   </joint>
-  <joint name="table_leg_FR_to_world" type="fixed">
-    <parent link="world"/>
+  <joint name="table_leg_FR_to_tabletop" type="fixed">
+    <parent link="tabletop"/>
     <child link="table_leg_FR"/>
-    <origin xyz="${3*table_inner_width/8} ${-3*table_inner_length/8} 0"/>
+    <origin xyz="${table_inner_width/2} ${-table_inner_length/2} 0"/>
   </joint>
-  <joint name="table_leg_BR_to_world" type="fixed">
-    <parent link="world"/>
+  <joint name="table_leg_BR_to_tabletop" type="fixed">
+    <parent link="tabletop"/>
     <child link="table_leg_BR"/>
-    <origin xyz="${-3*table_inner_width/8} ${-3*table_inner_length/8} 0"/>
+    <origin xyz="${-table_inner_width/2} ${-table_inner_length/2} 0"/>
   </joint>
-  <!-- Tabletop (CAD?)
-    <link name="
-  -->
+</robot>

Commit message: update pool_bot

File: URDF/pool_bot.xacro (robot description, xacro)
@@ -10,4 +10,6 @@
   <xacro:property name="table_inner_height" value="0.75"/>
   <xacro:property name="table_outer_height" value="0.8"/>
+  <xacro:property name="tabletop_inner_height" value="${table_inner_height-table_leg_length}"/>
+  <xacro:property name="tabletop_outer_height" value="${table_outer_height-table_leg_length}"/>
   <!-- Define macro for table legs -->
   <xacro:macro name="table_leg" params="name">
@@ -44,14 +46,14 @@
     <visual>
       <geometry>
-        <box size="${table_outer_width} ${table_outer_length} ${table_inner_height-table_leg_length}"/>
+        <box size="${table_outer_width} ${table_outer_length} ${tabletop_inner_height}"/>
       </geometry>
-      <origin xyz="0 0 ${(table_inner_height-table_leg_length)/2}"/>
+      <origin xyz="0 0 ${(tabletop_inner_height)/2}"/>
       <material name="brown"/>
     </visual>
     <collision>
       <geometry>
-        <box size="${table_outer_width} ${table_outer_length} ${table_inner_height-table_leg_length}"/>
+        <box size="${table_outer_width} ${table_outer_length} ${tabletop_inner_height}"/>
       </geometry>
-      <origin xyz="0 0 ${(table_inner_height-table_leg_length)/2}"/>
+      <origin xyz="0 0 ${(tabletop_inner_height)/2}"/>
     </collision>
   </link>
@@ -61,4 +63,5 @@
     <origin xyz="0 0 ${table_leg_length}"/>
   </joint>
+  <!-- table_frame_ends, table_frame_sides -->
   <xacro:table_leg name="FL"/>
   <xacro:table_leg name="BL"/>

Commit message: add Path object to reader.py

File: URDF/pool_bot.xacro (robot description, xacro)
@@ -40,4 +40,7 @@
     <color rgba="0.56 0.32 0.12 1"/>
   </material>
+  <material name="green">
+    <color rgba="0 1 0 1"/>
+  </material>
   <!-- Define links and joints -->
   <link name="world">
@@ -49,5 +52,5 @@
       </geometry>
       <origin xyz="0 0 ${(tabletop_inner_height)/2}"/>
-      <material name="brown"/>
+      <material name="green"/>
     </visual>
     <collision>
