Commit message: Start assignment bot model

File: URDF/MDaK_assignment_1.urdf (robot description, URDF)
Before this commit: robot myfirst, 16 links, 15 joints
Links:
- removed link base_link
- removed link box
- removed link gripper_pole
- removed link head
- removed link left_back_wheel
- removed link left_base
- removed link left_front_wheel
- removed link left_gripper
- removed link left_leg
- removed link left_tip
- removed link right_back_wheel
- removed link right_base
- removed link right_front_wheel
- removed link right_gripper
- removed link right_leg
- removed link right_tip
- added link base_box; collision box size=0.2 0.12 0.1; visual box size=0.2 0.12 0.1
- added link world
Joints:
- removed joint base_to_left_leg
- removed joint base_to_right_leg
- removed joint gripper_extension
- removed joint head_swivel
- removed joint left_back_wheel_joint
- removed joint left_base_joint
- removed joint left_front_wheel_joint
- removed joint left_gripper_joint
- removed joint left_tip_joint
- removed joint right_back_wheel_joint
- removed joint right_base_joint
- removed joint right_front_wheel_joint
- removed joint right_gripper_joint
- removed joint right_tip_joint
- removed joint tobox
- added joint base_box_to_world: type fixed, parent world, child base_box, origin xyz=0 0 0.05

Commit message: Model arm 1 on assignment bot

File: URDF/MDaK_assignment_1.urdf (robot description, URDF)
Before this commit: robot franka_research_3, 2 links, 1 joints
Links:
- added link arm_link_1a; collision cylinder length=0.14 radius=0.06; visual cylinder length=0.14 radius=0.06
- added link arm_link_1b; collision cylinder length=0.06 radius=0.06; visual cylinder length=0.06 radius=0.06
- added link arm_link_1c; collision sphere radius=0.06; visual sphere radius=0.06
- added link base_cyl; collision cylinder length=0.033 radius=0.065; visual cylinder length=0.033 radius=0.06
Joints:
- added joint arm_link_1a_to_1b: type fixed, parent arm_link_1a, child arm_link_1b, origin xyz=0 0 0.2
- added joint arm_link_1a_to_base: type revolute, parent base_cyl, child arm_link_1a, origin xyz=0 0 0.033, axis 0 0 1, limit lower=-2.897247 upper=2.897247 effort=1000.0 velocity=2.617994
- added joint arm_link_1b_to_1c: type fixed, parent arm_link_1b, child arm_link_1c, origin xyz=0 -0.06 0
- added joint base_cyl_to_base_box: type fixed, parent base_box, child base_cyl, origin xyz=0.04 0 0.1
- joint base_box_to_world: origin xyz=0 0 0.05 -> xyz=0 0 0

Commit message: Model up to arm 3 in assignment 1

File: URDF/MDaK_assignment_1.urdf (robot description, URDF)
Before this commit: robot franka_research_3, 6 links, 5 joints
Links:
- added link arm_link_2a; collision cylinder length=0.14 radius=0.06; visual cylinder length=0.14 radius=0.06
- added link arm_link_2b; collision cylinder length=0.06 radius=0.06; visual cylinder length=0.06 radius=0.06
- added link arm_link_2c; collision sphere radius=0.06; visual sphere radius=0.06
- added link arm_link_3a; collision cylinder length=0.05 radius=0.06; visual cylinder length=0.05 radius=0.06
- added link arm_link_3b; collision cylinder length=0.06 radius=0.06; visual cylinder length=0.06 radius=0.06
- added link arm_link_3c; collision sphere radius=0.06; visual sphere radius=0.06
- added link arm_link_3d; collision cylinder length=0.02 radius=0.06; visual cylinder length=0.02 radius=0.06
- added link arm_link_3e; collision sphere radius=0.05; visual sphere radius=0.05
Joints:
- removed joint arm_link_1a_to_1b
- removed joint arm_link_1a_to_base
- removed joint arm_link_1b_to_1c
- added joint arm_link_1a_to_base_cyl: type revolute, parent base_cyl, child arm_link_1a, origin xyz=0 0 0.033, axis 0 0 1, limit lower=-2.897247 upper=2.897247 effort=1000.0 velocity=2.617994
- added joint arm_link_1b_to_1a: type fixed, parent arm_link_1a, child arm_link_1b, origin xyz=0 0 0.2
- added joint arm_link_1c_to_1b: type fixed, parent arm_link_1b, child arm_link_1c, origin xyz=0 -0.06 0
- added joint arm_link_2a_to_2b: type fixed, parent arm_link_2b, child arm_link_2a, origin xyz=0 0 0.06
- added joint arm_link_2b_to_1b: type revolute, parent arm_link_1b, child arm_link_2b, origin xyz=0 0 0, axis 0 1 0, limit lower=-1.832596 upper=1.832596 effort=1000.0 velocity=2.617994
- added joint arm_link_2c_to_2b: type fixed, parent arm_link_2b, child arm_link_2c, origin xyz=0 0.06 0
- added joint arm_link_3a_to_2a: type revolute, parent arm_link_2a, child arm_link_3a, origin xyz=0 0 0.14, axis 0 0 1, limit lower=-2.897247 upper=2.897247 effort=1000.0 velocity=2.617994
- added joint arm_link_3b_to_3a: type fixed, parent arm_link_3a, child arm_link_3b, origin xyz=0.082 0 0.116
- added joint arm_link_3c_to_3a: type fixed, parent arm_link_3a, child arm_link_3c, origin xyz=0 0 0.06
- added joint arm_link_3d_to_3b: type fixed, parent arm_link_3b, child arm_link_3d, origin xyz=0 0.06 0
- added joint arm_link_3e_to_3b: type fixed, parent arm_link_3b, child arm_link_3e, origin xyz=0 0.06 0

File: URDF/tutorial1.urdf (robot description, URDF)
Before this commit: robot franka_research_3, 17 links, 16 joints
Links:
- removed link world
Joints:
- removed joint base_world_fix
- joint gripper_extension: axis 0 1 0 -> 1 0 0

Commit message: Model up to arm 4a in assignment

File: URDF/MDaK_assignment_1.urdf (robot description, URDF)
Before this commit: robot franka_research_3, 14 links, 13 joints
Links:
- added link arm_link_4a; collision cylinder length=0.05 radius=0.06; visual cylinder length=0.05 radius=0.06
- added link arm_link_4b; collision cylinder length=0.06 radius=0.06; visual cylinder length=0.06 radius=0.06
- added link arm_link_4c; collision sphere radius=0.06; visual sphere radius=0.06
Joints:
- added joint arm_link_4a_to_4b: type fixed, parent arm_link_4b, child arm_link_4a, origin xyz=0.116 0 0.082 rpy=0 0 0
- added joint arm_link_4b_to_3b: type revolute, parent arm_link_3b, child arm_link_4b, origin xyz=0 0 0 rpy=0 0 0, axis 0 1 0, limit lower=-1.448623 upper=1.500983 effort=1000.0 velocity=2.617994
- added joint arm_link_4c_to_4a: type fixed, parent arm_link_4a, child arm_link_4c, origin xyz=-0.06 0 0

Commit message: Add robot arm 5 in assignment 1

File: URDF/MDaK_assignment_1.urdf (robot description, URDF)
Before this commit: robot franka_research_3, 17 links, 16 joints
Links:
- added link arm_link_4d; collision cylinder length=0.02 radius=0.06; visual cylinder length=0.02 radius=0.06
- added link arm_link_4e; collision sphere radius=0.05; visual sphere radius=0.05
- added link arm_link_5a; collision cylinder length=0.208 radius=0.06; visual cylinder length=0.208 radius=0.06
- added link arm_link_5b; visual cylinder length=0.06 radius=0.06
Joints:
- added joint arm_link_4d_to_4b: type fixed, parent arm_link_4b, child arm_link_4d, origin xyz=0 -0.06 0
- added joint arm_link_4e_to_4b: type fixed, parent arm_link_4b, child arm_link_4e, origin xyz=0 -0.06 0
- added joint arm_link_5a_to_4a: type revolute, parent arm_link_4a, child arm_link_5a, origin xyz=0 0 0 rpy=0 0 0, axis 1 0 0, limit lower=-2.879793 upper=2.879793 effort=1000.0 velocity=5.253441
- added joint arm_link_5b_to_5a: type fixed, parent arm_link_5a, child arm_link_5b, origin xyz=0.268 0 0 rpy=0 0 0

Commit message: add shape to arm 5

File: URDF/MDaK_assignment_1.urdf (robot description, URDF)
Before this commit: robot franka_research_3, 21 links, 20 joints
Links:
- added link arm_link_5c; collision sphere radius=0.06; visual sphere radius=0.06
- added link arm_link_5d; collision cylinder length=0.168 radius=0.03; visual cylinder length=0.168 radius=0.03
- link arm_link_3a: geometry collision cylinder length=0.06 radius=0.06; visual cylinder length=0.06 radius=0.06
- link arm_link_4a: geometry collision cylinder length=0.06 radius=0.06; visual cylinder length=0.06 radius=0.06
- link arm_link_5a: geometry collision cylinder length=0.06 radius=0.06; visual cylinder length=0.06 radius=0.06
- link arm_link_5b: geometry collision cylinder length=0.06 radius=0.06; visual cylinder length=0.06 radius=0.06
Joints:
- added joint arm_link_5c_to_5a: type fixed, parent arm_link_5a, child arm_link_5c, origin xyz=0.06 0 0
- added joint arm_link_5d_to_5a: type fixed, parent arm_link_5a, child arm_link_5d, origin xyz=0.06 0 0 rpy=0 0 0

Commit message: begin link 6

File: URDF/MDaK_assignment_1.urdf (robot description, URDF)
Before this commit: robot franka_research_3, 23 links, 22 joints
Links:
- added link arm_link_6a; collision cylinder length=0.12 radius=0.06; visual cylinder length=0.12 radius=0.06
- added link arm_link_6b; collision cylinder length=0.06 radius=0.06; visual cylinder length=0.06 radius=0.06
Joints:
- added joint arm_link_6a_to_6b: type fixed
- added joint arm_link_6b_to_5b: type revolute, parent arm_link_5b, child arm_link_6b, origin xyz=0 0 0 rpy=0 0 0, axis 0 1 0, limit lower=-1.134464 upper=3.054326 effort=1000.0 velocity=5.253441

Commit message: finish arm model

File: URDF/MDaK_assignment_1.urdf (robot description, URDF)
Before this commit: robot franka_research_3, 25 links, 24 joints
Links:
- added link arm_link_6c; visual box size=0.088 0.03 0.08
- added link arm_link_7a; collision cylinder length=0.047 radius=0.045; visual cylinder length=0.047 radius=0.045
- added link arm_link_7b; visual cylinder length=0.01 radius=0.0325
- added link arm_link_7c; collision box size=0.09 0.0825 0.0375; visual box size=0.09 0.0825 0.0375
- link arm_link_5b: geometry collision cylinder length=0.06 radius=0.05; visual cylinder length=0.06 radius=0.05
- link arm_link_6a: geometry collision cylinder length=0.13 radius=0.045; visual cylinder length=0.13 radius=0.045
- link arm_link_6b: geometry collision cylinder length=0.06 radius=0.05; visual cylinder length=0.06 radius=0.05
Joints:
- added joint arm_link_6c_to_6b: type fixed, parent arm_link_6b, child arm_link_6c, origin xyz=0 -0.03 0 rpy=0 0 0.174533
- added joint arm_link_7a_to_6a: type revolute, parent arm_link_6a, child arm_link_7a, origin xyz=0 0 0 rpy=0 0 0, axis 0 0 1, limit lower=-3.054326 upper=3.054326 effort=1000.0 velocity=5.253441
- added joint arm_link_7b_to_7a: type fixed, parent arm_link_7a, child arm_link_7b, origin xyz=0 0 -0.057 rpy=0 0 0
- added joint arm_link_7c_to_7a: type fixed, parent arm_link_7a, child arm_link_7c, origin xyz=0 0 -0.047 rpy=0 0 -0.785398
- joint arm_link_6a_to_6b: child (none) -> arm_link_6a; origin (none) -> xyz=0.088 0.0 -0.045 rpy=0 0 0; parent (none) -> arm_link_6b

Commit message: add inertial tags to fr3, start to add jointMotorControls

File: URDF/MDaK_assignment_1.urdf (robot description, URDF)
Before this commit: robot franka_research_3, 29 links, 28 joints
Links:
- link arm_link_1a: mass None -> 3
- link arm_link_1b: mass None -> 0.1
- link arm_link_1c: mass None -> 0.1
- link arm_link_2a: mass None -> 3
- link arm_link_2b: mass None -> 0.1
- link arm_link_2c: mass None -> 0.1
- link arm_link_3a: mass None -> 3
- link arm_link_3b: mass None -> 0.1
- link arm_link_3c: mass None -> 0.1
- link arm_link_3d: mass None -> 0.1
- link arm_link_3e: mass None -> 0.1
- link arm_link_4a: mass None -> 3
- link arm_link_4b: mass None -> 0.1
- link arm_link_4c: mass None -> 0.1
- link arm_link_4d: mass None -> 0.1
- link arm_link_4e: mass None -> 0.1
- link arm_link_5a: mass None -> 2
- link arm_link_5b: mass None -> 0.1
- link arm_link_5c: mass None -> 0.1
- link arm_link_5d: mass None -> 0.1
- link arm_link_6a: mass None -> 1
- link arm_link_6b: mass None -> 0.1
- link arm_link_6c: mass None -> 0.1; geometry collision box size=0.088 0.03 0.08; visual box size=0.088 0.03 0.08
- link arm_link_7a: mass None -> 0.3
- link arm_link_7b: mass None -> 0.1; geometry collision cylinder length=0.01 radius=0.0325; visual cylinder length=0.01 radius=0.0325
- link arm_link_7c: mass None -> 0.1
- link base_box: mass None -> 2.5
- link base_cyl: mass None -> 0.1
