Commit message: Update Ass4, finish pool-bot

File: Assignment/pool_bot.urdf (robot description, URDF)
Before this commit: robot pool_table, 6 links, 5 joints
Links:
- added link bot_leg_BL; collision box size=0.05 0.05 0.15; visual box size=0.05 0.05 0.15
- added link bot_leg_BR; collision box size=0.05 0.05 0.15; visual box size=0.05 0.05 0.15
- added link bot_leg_FL; collision box size=0.05 0.05 0.15; visual box size=0.05 0.05 0.15
- added link bot_leg_FR; collision box size=0.05 0.05 0.15; visual box size=0.05 0.05 0.15
- added link head; collision box size=0.1 .1 .2; visual box size=0.1 .1 .1
- added link rail_l_B; collision box size=0.05 1.7999999999999998 0.05; visual box size=0.05 1.7999999999999998 0.05
- added link rail_l_F; collision box size=0.05 1.7999999999999998 0.05; visual box size=0.05 1.7999999999999998 0.05
- added link rail_w; collision box size=1.02 0.05 0.05; visual box size=1.02 0.05 0.05
- added link rail_z; collision box size=0.05 0.05 .2; visual box size=0.05 0.05 .2
- added link table_end_B; collision box size=1.12 0.1499999999999999 0.050000000000000044; visual box size=1.12 0.1499999999999999 0.050000000000000044
- added link table_end_F; collision box size=1.12 0.1499999999999999 0.050000000000000044; visual box size=1.12 0.1499999999999999 0.050000000000000044
- added link table_side_L; collision box size=0.15000000000000008 1.6 0.050000000000000044; visual box size=0.15000000000000008 1.6 0.050000000000000044
- added link table_side_R; collision box size=0.15000000000000008 1.6 0.050000000000000044; visual box size=0.15000000000000008 1.6 0.050000000000000044
Joints:
- added joint bot_leg_BL_to_tabletop: type fixed, parent tabletop, child bot_leg_BL, origin xyz=-0.535 0.9249999999999999 0.30000000000000004
- added joint bot_leg_BR_to_tabletop: type fixed, parent tabletop, child bot_leg_BR, origin xyz=-0.535 -0.9249999999999999 0.30000000000000004
- added joint bot_leg_FL_to_tabletop: type fixed, parent tabletop, child bot_leg_FL, origin xyz=0.535 0.9249999999999999 0.30000000000000004
- added joint bot_leg_FR_to_tabletop: type fixed, parent tabletop, child bot_leg_FR, origin xyz=0.535 -0.9249999999999999 0.30000000000000004
- added joint head_to_rail_w: type prismatic, parent rail_w, child head, origin xyz=0 0.05 0, axis 1 0 0, limit lower=-0.48500000000000004 upper=0.48500000000000004 effort=1000.0 velocity=5
- added joint rail_l_B_to_bot_leg_BL: type fixed, parent bot_leg_BL, child rail_l_B, origin xyz=0 -0.9249999999999999 0.15
- added joint rail_l_F_to_bot_leg_FL: type fixed, parent bot_leg_FL, child rail_l_F, origin xyz=0 -0.9249999999999999 0.15
- added joint rail_w_to_rail_l_F: type prismatic, parent rail_l_F, child rail_w, origin xyz=-0.535 0 0, axis 0 1 0, limit lower=-0.8999999999999999 upper=0.8999999999999999 effort=1000.0 velocity=5
- added joint rail_z_to_head: type prismatic, parent head, child rail_z, origin xyz=0 0 -0.1, axis 0 0 -1, limit lower=0 upper=0.1 effort=1000.0 velocity=5
- added joint table_end_B_to_tabletop: type fixed, parent tabletop, child table_end_B, origin xyz=0 0.875 0.25
- added joint table_end_F_to_tabletop: type fixed, parent tabletop, child table_end_F, origin xyz=0 -0.875 0.25
- added joint table_side_L_to_tabletop: type fixed, parent tabletop, child table_side_L, origin xyz=-0.485 0 0.25
- added joint table_side_R_to_tabletop: type fixed, parent tabletop, child table_side_R, origin xyz=0.485 0 0.25

File: Assignment/pool_bot.xacro (robot description, xacro)
@@ -1,4 +1,21 @@
 <?xml version="1.0"?>
 <robot xmlns:xacro="http://www.ros.org/wiki/xacro" name="pool_table">
+  <!-- Define Materials -->
+  <material name="black">
+    <color rgba="0 0 0 1"/>
+  </material>
+  <material name="grey">
+    <color rgba="0.75 0.75 0.75 1"/>
+  </material>
+  <material name="white">
+    <color rgba="1 1 1 1"/>
+  </material>
+  <material name="brown">
+    <color rgba="0.56 0.32 0.12 1"/>
+  </material>
+  <material name="green">
+    <color rgba="0 0.5 0 1"/>
+  </material>
+  <!-- Table -->
   <!-- Define Parameters -->
   <xacro:property name="table_leg_radius" value="0.075"/>
@@ -30,17 +47,39 @@
     </link>
   </xacro:macro>
-  <!-- Define Materials -->
-  <material name="black">
-    <color rgba="0 0 0 1"/>
-  </material>
-  <material name="white">
-    <color rgba="1 1 1 1"/>
-  </material>
-  <material name="brown">
-    <color rgba="0.56 0.32 0.12 1"/>
-  </material>
-  <material name="green">
-    <color rgba="0 0.5 0 1"/>
-  </material>
+  <!-- Define macro for table edges -->
+  <xacro:macro name="table_end" params="name">
+    <link name="table_end_${name}">
+      <visual>
+        <geometry>
+          <box size="${table_outer_width} ${(table_outer_length-table_inner_length)/2} ${table_outer_height-table_inner_height}"/>
+        </geometry>
+        <origin xyz="0 0 ${(table_outer_height-table_inner_height)/2}"/>
+        <material name="green"/>
+      </visual>
+      <collision>
+        <geometry>
+          <box size="${table_outer_width} ${(table_outer_length-table_inner_length)/2} ${table_outer_height-table_inner_height}"/>
+        </geometry>
+      </collision>
+      <origin xyz="0 0 ${(table_outer_height-table_inner_height)/2}"/>
+    </link>
+  </xacro:macro>
+    <xacro:macro name="table_side" params="name">
+    <link name="table_side_${name}">
+      <visual>
+        <geometry>
+          <box size="${(table_outer_width-table_inner_width)/2} ${table_inner_length} ${table_outer_height-table_inner_height}"/>
+        </geometry>
+        <origin xyz="0 0 ${(table_outer_height-table_inner_height)/2}"/>
+        <material name="green"/>
+      </visual>
+      <collision>
+        <geometry>
+          <box size="${(table_outer_width-table_inner_width)/2} ${table_inner_length} ${table_outer_height-table_inner_height}"/>
+        </geometry>
+      </collision>
+      <origin xyz="0 0 ${(table_outer_height-table_inner_height)/2}"/>
+    </link>
+  </xacro:macro>
   <!-- Define links and joints -->
   <link name="world">
@@ -66,5 +105,4 @@
     <origin xyz="0 0 ${table_leg_length}"/>
   </joint>
-  <!-- table_frame_ends, table_frame_sides -->
   <xacro:table_leg name="FL"/>
   <xacro:table_leg name="BL"/>
@@ -91,3 +129,172 @@
     <origin xyz="${-table_inner_width/2} ${-table_inner_length/2} 0"/>
   </joint>
+  <xacro:table_end name="F"/>
+  <xacro:table_end name="B"/>
+  <xacro:table_side name="L"/>
+  <xacro:table_side name="R"/>
+  <joint name="table_end_F_to_tabletop" type="fixed">
+    <parent link="tabletop"/>
+    <child link="table_end_F"/>
+    <origin xyz="0 -${(table_outer_length-(table_outer_length-table_inner_length)/2)/2} ${tabletop_inner_height}"/>
+  </joint>
+  <joint name="table_end_B_to_tabletop" type="fixed">
+    <parent link="tabletop"/>
+    <child link="table_end_B"/>
+    <origin xyz="0 ${(table_outer_length-(table_outer_length-table_inner_length)/2)/2} ${tabletop_inner_height}"/>
+  </joint>
+  <joint name="table_side_L_to_tabletop" type="fixed">
+    <parent link="tabletop"/>
+    <child link="table_side_L"/>
+    <origin xyz="-${(table_outer_width-(table_outer_width-table_inner_width)/2)/2} 0 ${tabletop_inner_height}"/>
+  </joint>
+  <joint name="table_side_R_to_tabletop" type="fixed">
+    <parent link="tabletop"/>
+    <child link="table_side_R"/>
+    <origin xyz="${(table_outer_width-(table_outer_width-table_inner_width)/2)/2} 0 ${tabletop_inner_height}"/>
+  </joint>
+  <!-- Robot -->
+  <!-- Define Parameters for robot -->
+  <!-- Define Parameters -->
+  <xacro:property name="bot_leg_width" value="0.05"/>
+  <xacro:property name="bot_leg_height" value="0.15"/>
+  <xacro:property name="bot_length" value="${table_outer_length-bot_leg_width}"/>
+  <xacro:property name="bot_width" value="${table_outer_width-bot_leg_width}"/>
+  <!-- Define Macros for robot -->
+  <xacro:macro name="bot_leg" params="name">
+    <link name="bot_leg_${name}">
+      <visual>
+        <geometry>
+          <box size="${bot_leg_width} ${bot_leg_width} ${bot_leg_height}"/>
+        </geometry>
+        <origin xyz="0 0 0.075"/>
+        <material name="grey"/>
+      </visual>
+      <collision>
+        <geometry>
+          <box size="${bot_leg_width} ${bot_leg_width} ${bot_leg_height}"/>
+        </geometry>
+        <origin xyz="0 0 ${bot_leg_height/2}"/>
+      </collision>
+    </link>
+  </xacro:macro>
+    <xacro:macro name="rail_l" params="name">
+    <link name="rail_l_${name}">
+      <visual>
+        <geometry>
+          <box size="${bot_leg_width} ${bot_length-bot_leg_width} ${bot_leg_width}"/>
+        </geometry>
+        <origin xyz="0 0 -${bot_leg_width/2}"/>
+        <material name="grey"/>
+      </visual>
+      <collision>
+        <geometry>
+          <box size="${bot_leg_width} ${bot_length-bot_leg_width} ${bot_leg_width}"/>
+        </geometry>
+        <origin xyz="0 0 -${bot_leg_width/2}"/>
+      </collision>
+    </link>
+  </xacro:macro>
+  <!-- Define Links and Joints for robot -->
+  <xacro:bot_leg name="FL"/>
+  <xacro:bot_leg name="BL"/>
+  <xacro:bot_leg name="FR"/>
+  <xacro:bot_leg name="BR"/>
+  <joint name="bot_leg_FL_to_tabletop" type="fixed">
+    <parent link="tabletop"/>
+    <child link="bot_leg_FL"/>
+    <origin xyz="${bot_width/2} ${(bot_length)/2} ${tabletop_outer_height}"/>
+  </joint>
+    <joint name="bot_leg_BL_to_tabletop" type="fixed">
+    <parent link="tabletop"/>
+    <child link="bot_leg_BL"/>
+    <origin xyz="-${bot_width/2} ${(bot_length)/2} ${tabletop_outer_height}"/>
+  </joint>
+  <joint name="bot_leg_FR_to_tabletop" type="fixed">
+    <parent link="tabletop"/>
+    <child link="bot_leg_FR"/>
+    <origin xyz="${bot_width/2} -${(bot_length)/2} ${tabletop_outer_height}"/>
+  </joint>
+  <joint name="bot_leg_BR_to_tabletop" type="fixed">
+    <parent link="tabletop"/>
+    <child link="bot_leg_BR"/>
+    <origin xyz="-${bot_width/2} -${(bot_length)/2} ${tabletop_outer_height}"/>
+  </joint>
+  <xacro:rail_l name="F"/>
+  <xacro:rail_l name="B"/>
+  <joint name="rail_l_F_to_bot_leg_FL" type="fixed">
+    <parent link="bot_leg_FL"/>
+    <child link="rail_l_F"/>
+    <origin xyz="0 -${bot_length/2} ${bot_leg_height}"/>
+  </joint>
+  <joint name="rail_l_B_to_bot_leg_BL" type="fixed">
+    <parent link="bot_leg_BL"/>
+    <child link="rail_l_B"/>
+    <origin xyz="0 -${bot_length/2} ${bot_leg_height}"/>
+  </joint>
+  <link name="rail_w">
+    <visual>
+      <geometry>
+        <box size="${bot_width-bot_leg_width} ${bot_leg_width} ${bot_leg_width}"/>
+      </geometry>
+      <origin xyz="0 0 -${bot_leg_width/2}"/>
+      <material name="grey"/>
+    </visual>
+    <collision>
+      <geometry>
+        <box size="${bot_width-bot_leg_width} ${bot_leg_width} ${bot_leg_width}"/>
+      </geometry>
+      <origin xyz="0 0 -${bot_leg_width/2}"/>
+    </collision>
+  </link>
+  <joint name="rail_w_to_rail_l_F" type="prismatic">
+    <parent link="rail_l_F"/>
+    <child link="rail_w"/>
+    <origin xyz="-${(bot_width)/2} 0 0"/>
+    <limit effort="1000.0" lower="-${(bot_length-bot_leg_width)/2}" upper="${(bot_length-bot_leg_width)/2}" velocity="5"/>
+    <axis xyz="0 1 0"/>
+  </joint>
+  <link name="head">
+    <visual>
+      <geometry>
+        <box size="0.1 .1 .1"/>
+      </geometry>
+      <origin xyz="0 0 0"/>
+      <material name="grey"/>
+    </visual>
+    <collision>
+      <geometry>
+        <box size="0.1 .1 .2"/>
+      </geometry>
+      <origin xyz="0 0 0"/>
+    </collision>
+  </link>
+  <joint name="head_to_rail_w" type="prismatic">
+    <parent link="rail_w"/>
+    <child link="head"/>
+    <origin xyz="0 ${bot_leg_width} 0"/>
+    <axis xyz="1 0 0"/>
+    <limit effort="1000.0" lower="-${(bot_width/2)-bot_leg_width}" upper="${(bot_width/2)-bot_leg_width}" velocity="5"/>
+  </joint>
+  <link name="rail_z">
+    <visual>
+      <geometry>
+        <box size="${bot_leg_width} ${bot_leg_width} .2"/>
+      </geometry>
+      <origin xyz="0 0 0.1"/>
+      <material name="grey"/>
+    </visual>
+    <collision>
+       <geometry>
+        <box size="${bot_leg_width} ${bot_leg_width} .2"/>
+      </geometry>
+      <origin xyz="0 0 0.1"/>
+    </collision>
+  </link>
+  <joint name="rail_z_to_head" type="prismatic">
+    <parent link="head"/>
+    <child link="rail_z"/>
+    <origin xyz="0 0 -0.1"/>
+    <axis xyz="0 0 -1"/>
+    <limit effort="1000.0" lower="0" upper="0.1" velocity="5"/>
+  </joint>
 </robot>
